Commit message: Add files via upload

File: robot.urdf (robot description, URDF)
Before this commit: robot robot, 6 links, 5 joints
Links:
- removed link axis_Link
- removed link front_Link
- removed link left_Link
- removed link right_Link
- added link back_left_Link, mass 0.58827061564709; collision mesh filename=package://robot/meshes/back_left_Link.STL; visual mesh filename=package://robot/meshes/back_left_Link.STL
- added link back_right_Link, mass 0.588270615647089; collision mesh filename=package://robot/meshes/back_right_Link.STL; visual mesh filename=package://robot/meshes/back_right_Link.STL
- added link front_left_Link, mass 0.588270615647091; collision mesh filename=package://robot/meshes/front_left_Link.STL; visual mesh filename=package://robot/meshes/front_left_Link.STL
- added link front_right_Link, mass 0.58827061564709; collision mesh filename=package://robot/meshes/front_right_Link.STL; visual mesh filename=package://robot/meshes/front_right_Link.STL
- added link laser_Link, mass 0.0296109461913993; collision mesh filename=package://robot/meshes/laser_Link.STL; visual mesh filename=package://robot/meshes/laser_Link.STL
- link base_link: mass 40.4999492858241 -> 43.7289793607304
Joints:
- removed joint axis
- removed joint front
- removed joint left
- removed joint right
- added joint back_left: type continuous, parent base_link, child back_left_Link, origin xyz=-0.135 0.15 0.069 rpy=1.5708 0 0, axis 0 0 1
- added joint back_right: type continuous, parent base_link, child back_right_Link, origin xyz=-0.135 -0.15 0.069 rpy=-1.5708 0 0, axis 0 0 1
- added joint front_left: type continuous, parent base_link, child front_left_Link, origin xyz=0.155 0.15 0.069 rpy=1.5708 0 0, axis 0 0 -1
- added joint front_right: type continuous, parent base_link, child front_right_Link, origin xyz=0.155 -0.15 0.069 rpy=-1.5708 0 0, axis 0 0 -1
- added joint laser: type fixed, parent base_link, child laser_Link, origin xyz=0.205 0 0.156 rpy=0 0 0, axis 0 0 0
- joint kinect: origin xyz=0.185 0 0.297 rpy=0 0 0 -> xyz=0.185 0 0.207 rpy=0 0 0
